File: separator_pcb/Separator.kicad_sch (KiCad schematic)
At the start: 10 parts, among them J1 L_COL_CONN, Q1 BSS138

Commit message: Footprint placement done, PWR needs connecting
Parts:
- J1: value L_COL_CONN -> COL_CONN; footprint Connector_PinHeader_1.00mm:PinHeader_2x02_P1.00mm_Vertical -> Connector_PinHeader_2.00mm:PinHeader_2x02_P2.00mm_Vertical
Changed lines of the file:
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@@
 			)
 		)
-		(property "Value" "L_COL_CONN"
+		(property "Value" "COL_CONN"
 			(at 152.4 119.38 0)
 			(effects
@@
 			)
 		)
-		(property "Footprint" "Connector_PinHeader_1.00mm:PinHeader_2x02_P1.00mm_Vertical"
+		(property "Footprint" "Connector_PinHeader_2.00mm:PinHeader_2x02_P2.00mm_Vertical"
 			(at 151.13 123.19 0)
 			(effects

Commit message: Layout done, generated fabrication files
Connections:
- net GND: now also H1.1, H2.1
- no-connect marks 3 -> 1
Other:
- moved on the sheet: H2
Changed lines of the file:
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@@
-	)
-	(no_connect
-		(at 224.79 22.86)
 	)
 	(no_connect
 		(at 185.42 96.52)
-	)
-	(no_connect
-		(at 224.79 30.48)
 	)
 	(wire
@@
 	(symbol
 		(lib_id "power:GND")
+		(at 224.79 22.86 0)
+		(unit 1)
+		(exclude_from_sim no)
+		(in_bom yes)
+		(on_board yes)
+		(dnp no)
+		(fields_autoplaced yes)
+		(property "Reference" "#PWR016"
+			(at 224.79 29.21 0)
+			(effects
+				(font
+					(size 1.27 1.27)
+				)
+				(hide yes)
+			)
+		)
+		(property "Value" "GND"
+			(at 224.79 27.94 0)
+			(effects
+				(font
+					(size 1.27 1.27)
+				)
+			)
+		)
+		(property "Footprint" ""
+			(at 224.79 22.86 0)
+			(effects
+				(font
+					(size 1.27 1.27)
+				)
+				(hide yes)
+			)
+		)
+		(property "Datasheet" ""
+			(at 224.79 22.86 0)
+			(effects
+				(font
+					(size 1.27 1.27)
+				)
+				(hide yes)
+			)
+		)
+		(property "Description" "Power symbol creates a global label with name \"GND\" , ground"
+			(at 224.79 22.86 0)
+			(effects
+				(font
+					(size 1.27 1.27)
+				)
+				(hide yes)
+			)
+		)
+		(pin "1"
+		)
+		(instances
+			(project "Separator"
+				(path "/34951e98-25fa-4bcc-a56f-5aa93e8633e9"
+					(reference "#PWR016")
+					(unit 1)
+				)
+			)
+		)
+	)
+	(symbol
+		(lib_id "power:GND")
 		(at 251.46 22.86 0)
 		(unit 1)
@@
 	(symbol
 		(lib_id "Mechanical:MountingHole_Pad")
-		(at 224.79 27.94 0)
+		(at 224.79 33.02 0)
 		(unit 1)
 		(exclude_from_sim yes)
@@
 		(fields_autoplaced yes)
 		(property "Reference" "H2"
-			(at 227.33 25.3999 0)
+			(at 227.33 30.4799 0)
 			(effects
 				(font
@@
 		)
 		(property "Value" "MountingHole_Pad"
-			(at 227.33 27.9399 0)
+			(at 227.33 33.0199 0)
 			(effects
 				(font
@@
 		)
 		(property "Footprint" "MountingHole:MountingHole_3.2mm_M3_ISO14580_Pad_TopBottom"
-			(at 224.79 27.94 0)
+			(at 224.79 33.02 0)
 			(effects
 				(font
@@
 		)
 		(property "Datasheet" "~"
-			(at 224.79 27.94 0)
+			(at 224.79 33.02 0)
 			(effects
 				(font
@@
 		)
 		(property "Description" "Mounting Hole with connection"
-			(at 224.79 27.94 0)
+			(at 224.79 33.02 0)
 			(effects
 				(font
@@
 					(unit 1)
 				)
+			)
+		)
+	)
+	(symbol
+		(lib_id "power:GND")
+		(at 224.79 35.56 0)
+		(unit 1)
+		(exclude_from_sim no)
+		(in_bom yes)
+		(on_board yes)
+		(dnp no)
+		(fields_autoplaced yes)
+		(property "Reference" "#PWR015"
+			(at 224.79 41.91 0)
+			(effects
+				(font
+					(size 1.27 1.27)
+				)
+				(hide yes)
+			)
+		)
+		(property "Value" "GND"
+			(at 224.79 40.64 0)
+			(effects
+				(font
+					(size 1.27 1.27)
+				)
+			)
+		)
+		(property "Footprint" ""
+			(at 224.79 35.56 0)
+			(effects
+				(font
+					(size 1.27 1.27)
+				)
+				(hide yes)
+			)
+		)
+		(property "Datasheet" ""
+			(at 224.79 35.56 0)
+			(effects
+				(font
+					(size 1.27 1.27)
+				)
+				(hide yes)
+			)
+		)
+		(property "Description" "Power symbol creates a global label with name \"GND\" , ground"
+			(at 224.79 35.56 0)
+			(effects
+				(font
+					(size 1.27 1.27)
+				)
+				(hide yes)
+			)
+		)
+		(pin "1"
+		)
+		(instances
+			(project "Separator"
+				(path "/34951e98-25fa-4bcc-a56f-5aa93e8633e9"
+					(reference "#PWR015")
+					(unit 1)
+				)
