File: pcb/VFDClock.kicad_pcb (KiCad board)
At the start: 4 copper layers, 80 x 52.7 mm, 84 parts, among them J1 Conn_01x04_Socket, J2 R_SIG_CONN, J3 R_PWR_CONN, J4 USB_C_Receptacle_USB2.0_16P, J5 L_SIG_CONN, J6 L_PWR_CONN, J7 CONN_GPIO, J8 L_COL_CONN, J9 R_COL_CONN, SW1 SW_SPST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

Commit message: Replaced capacitor footprints with EIA-3216
Parts:
- C19, C7: footprint Capacitor_Tantalum_SMD:CP_EIA-3528-15_AVX-H -> Capacitor_Tantalum_SMD:CP_EIA-3216-18_Kemet-A
