File: pcb/VFDClock.kicad_sch (KiCad schematic)
At the start: 84 parts, among them J1 Conn_01x04_Socket, J2 R_SIG_CONN, J3 R_PWR_CONN, J4 USB_C_Receptacle_USB2.0_16P, J5 L_SIG_CONN, J6 L_PWR_CONN, J7 CONN_GPIO, J8 L_COL_CONN, J9 R_COL_CONN, SW1 SW_SPST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

Commit message: Replaced capacitor footprints with EIA-3216
Parts:
- C19, C7: footprint Capacitor_Tantalum_SMD:CP_EIA-3528-15_AVX-H -> Capacitor_Tantalum_SMD:CP_EIA-3216-18_Kemet-A
Changed lines of the file:
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@@
 			"AAAAAAAAAAAAAAAAAAAAAAAAAAAAAAAAAAAAAAAAAAAAAAAAAAAAAAAAAAAAAAAAAAAAAAAAAAAA"
 			"AAAAAAAAAAAAAAAAAAAAAAAAAAAAAAAAAAAAAAAAAAAAAAAAAAAAAAAAAAAAAAAAAAAAAAAAAAAA"
-			"AAAAAAAAAAAAAAAAAAAAAAAAAAAAAA=="
+			"AAAAAAAAAAAAAAAAAAAAAAAAAAAAAABPAHQAbgB5AGgAZQB5ADUATgBNAHAAZABjAEIAQwAwAEEA"
+			"SgBoAFEAQQBBAFIASwBBAGkASQBBAGcAQQBsAFcAUwBSAGkAcABSAHcAUQB4AGsATwBoADgATwBw"
+			"AHYAeABBAGkAZwBNAGkAZwBsAEIAQwBCAFUAbABCAEEASgBnAEMAaABNAHEARQBTAEkAVgBSAFUA"
+			"bQB5ADEAaQBrAHkAWQB0AEcAMABlADAASQA0AEsATwBVAGoALwByAEUAaQB3AG8AQgBSAEYAWQAr"
+			"AFYAVgBZAFUAOQBzADkASwBPADUAWABQADMAYQBpAHQAagB0AGkAZABKAGIALwBjAGUAMQBUAEUA"
+			"QQAzAGEAcgB2AFgAeQBvAGkAaQBsAHMAaABlAEYAWgBEAEkAegBNAHIANwBhAHUAZgBQAGMAMgBi"
+			"AE0AWABjAG4ATgBaAFMAMgBSAFUAVgBPAGUAdQBYAFMAWgBNAG4ATgBTADgAUgBRAHYASABlAEcA"
+			"VgBxADQAWQBpAHIAQQA5AGsAaAA3AHkAVQBsADkAWABCADIAcgBEAEkAYgBVAGEAWgBEAGsAVgBG"
+			"AFIAMABXADMAYQBqAEIAZwA1ADAAbQBrADgAWQA5AC8AZQB2AFoAOQAvADkAaABrADcASgBDAHcA"
+			"OAB2AEcAZgB2AFgAdABOAG4AUAB1ADAANABkAHcASgB3AEkAaQBkAG4ANwBhAHAAVgB0AGwATwBS"
+			"AHgAQgBrAHoAbgBGADYAYQBnAHMAVgBpADgAZgBlAC8AMwBjAFoAZAAvADQAdQBiACsATgByAGgA"
+			"bQArAFAAYQA4AFQAMgByAEIAUABkAGQAVwBkAGIAaQByAGwAcAAvADIAUwA0AG4ASABjAEQAVwB2"
+			"ADEAKwB4AGYAVwByAHIALwBhAEwAWQB6AHQAagB5AHkAMABWAC8AVwA3AFYAOQA2AG8AQgBiADQA"
+			"LwA1AFkAMABpAHIAYwB3AGgAeABtAFYAdQB4AHQAdwBFADYAUgBmAGwASwB6ACsAWABDAHcANwBU"
+			"AEEAYwB1AFcAawBRAHgAbgA3AFEAOQBOAHgAVgA2ADIAMQBSAGQAQgBQAHoAKwAvADkAWABGADIA"
+			"bwA3AEEATABrAGMAKwBsACsANAA0AE0ANwBoAGMAUAA3AEgANABaAGwAZgBIAEkANgBWAEMAbQBl"
+			"ADUAMABvADUAawBIAE4AZwBMAEkASAA3ADgARgBQADgAQQB6AGEAMABiAFIAUQBmADIANwBLAGoA"
+			"VwBXAFEASwBEAGQATgAxADcARABYAHoANQAzAGQAWABkAGUAZwAwAEEAOABPAFgANgBGAFcAVwBs"
+			"AHQANwBtAFgAYgBQAHQAawBkAFUASA=="
 		)
 	)
@@
 			)
 		)
-		(property "Footprint" "Capacitor_Tantalum_SMD:CP_EIA-3528-15_AVX-H"
+		(property "Footprint" "Capacitor_Tantalum_SMD:CP_EIA-3216-18_Kemet-A"
 			(at 58.1152 240.03 0)
 			(effects
@@
 			)
 		)
-		(property "Footprint" "Capacitor_Tantalum_SMD:CP_EIA-3528-15_AVX-H"
+		(property "Footprint" "Capacitor_Tantalum_SMD:CP_EIA-3216-18_Kemet-A"
 			(at 56.8452 180.34 0)
 			(effects
