File: module_pcb/Module.kicad_sch (KiCad schematic)
At the start: 29 parts, among them J1 L_SIG_CONN, J2 R_PWR_CONN, J3 R_SIG_CONN, J4 L_PWR_CONN, U1 AMS1117-3.3, U2 TBD62783AFNG, U3 SN74HC595PWR, U4 AMS1117-1.5

Commit message: Layout done
Parts:
- removed H4: MountingHole_Pad, MountingHole:MountingHole_3.2mm_M3_ISO14580_Pad_TopBottom, symbol Mechanical:MountingHole_Pad
Other:
- moved on the sheet: H1, H2, H3
Changed lines of the file:
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@@
 	(symbol
 		(lib_id "power:GND")
-		(at 236.22 38.1 0)
+		(at 217.17 38.1 0)
 		(unit 1)
 		(exclude_from_sim no)
@@
 		(fields_autoplaced yes)
 		(property "Reference" "#PWR08"
-			(at 236.22 44.45 0)
+			(at 217.17 44.45 0)
 			(effects
 				(font
@@
 		)
 		(property "Value" "GND"
-			(at 236.22 43.18 0)
+			(at 217.17 43.18 0)
 			(effects
 				(font
@@
 		)
 		(property "Footprint" ""
-			(at 236.22 38.1 0)
+			(at 217.17 38.1 0)
 			(effects
 				(font
@@
 		)
 		(property "Datasheet" ""
-			(at 236.22 38.1 0)
+			(at 217.17 38.1 0)
 			(effects
 				(font
@@
 		)
 		(property "Description" "Power symbol creates a global label with name \"GND\" , ground"
-			(at 236.22 38.1 0)
+			(at 217.17 38.1 0)
 			(effects
 				(font
@@
 	)
 	(symbol
-		(lib_id "Mechanical:MountingHole_Pad")
-		(at 259.08 48.26 0)
-		(unit 1)
-		(exclude_from_sim yes)
-		(in_bom no)
-		(on_board yes)
-		(dnp no)
-		(fields_autoplaced yes)
-		(property "Reference" "H4"
-			(at 261.62 45.7199 0)
-			(effects
-				(font
-					(size 1.27 1.27)
-				)
-				(justify left)
-			)
-		)
-		(property "Value" "MountingHole_Pad"
-			(at 261.62 48.2599 0)
-			(effects
-				(font
-					(size 1.27 1.27)
-				)
-				(justify left)
-			)
-		)
-		(property "Footprint" "MountingHole:MountingHole_3.2mm_M3_ISO14580_Pad_TopBottom"
-			(at 259.08 48.26 0)
-			(effects
-				(font
-					(size 1.27 1.27)
-				)
-				(hide yes)
-			)
-		)
-		(property "Datasheet" "~"
-			(at 259.08 48.26 0)
-			(effects
-				(font
-					(size 1.27 1.27)
-				)
-				(hide yes)
-			)
-		)
-		(property "Description" "Mounting Hole with connection"
-			(at 259.08 48.26 0)
-			(effects
-				(font
-					(size 1.27 1.27)
-				)
-				(hide yes)
-			)
-		)
-		(pin "1"
-		)
-		(instances
-			(project "Module"
-				(path "/34951e98-25fa-4bcc-a56f-5aa93e8633e9"
-					(reference "H4")
-					(unit 1)
-				)
-			)
-		)
-	)
-	(symbol
 		(lib_id "VFDClock_custom_lib:IV-22_VFD_Tube")
 		(at 110.49 137.16 90)
@@
 	(symbol
 		(lib_id "Mechanical:MountingHole_Pad")
-		(at 236.22 48.26 0)
+		(at 262.89 35.56 0)
 		(unit 1)
 		(exclude_from_sim yes)
@@
 		(fields_autoplaced yes)
 		(property "Reference" "H3"
-			(at 238.76 45.7199 0)
+			(at 265.43 33.0199 0)
 			(effects
 				(font
@@
 		)
 		(property "Value" "MountingHole_Pad"
-			(at 238.76 48.2599 0)
+			(at 265.43 35.5599 0)
 			(effects
 				(font
@@
 		)
 		(property "Footprint" "MountingHole:MountingHole_3.2mm_M3_ISO14580_Pad_TopBottom"
-			(at 236.22 48.26 0)
+			(at 262.89 35.56 0)
 			(effects
 				(font
@@
 		)
 		(property "Datasheet" "~"
-			(at 236.22 48.26 0)
+			(at 262.89 35.56 0)
 			(effects
 				(font
@@
 		)
 		(property "Description" "Mounting Hole with connection"
-			(at 236.22 48.26 0)
+			(at 262.89 35.56 0)
 			(effects
 				(font
@@
 	(symbol
 		(lib_id "power:GND")
-		(at 236.22 50.8 0)
+		(at 262.89 38.1 0)
 		(unit 1)
 		(exclude_from_sim no)
@@
 		(fields_autoplaced yes)
 		(property "Reference" "#PWR011"
-			(at 236.22 57.15 0)
+			(at 262.89 44.45 0)
 			(effects
 				(font
@@
 		)
 		(property "Value" "GND"
-			(at 236.22 55.88 0)
+			(at 262.89 43.18 0)
 			(effects
 				(font
@@
 		)
 		(property "Footprint" ""
-			(at 236.22 50.8 0)
+			(at 262.89 38.1 0)
 			(effects
 				(font
@@
 		)
 		(property "Datasheet" ""
-			(at 236.22 50.8 0)
+			(at 262.89 38.1 0)
 			(effects
 				(font
@@
 		)
 		(property "Description" "Power symbol creates a global label with name \"GND\" , ground"
-			(at 236.22 50.8 0)
+			(at 262.89 38.1 0)
 			(effects
 				(font
@@
 	(symbol
 		(lib_id "Mechanical:MountingHole_Pad")
-		(at 236.22 35.56 0)
+		(at 217.17 35.56 0)
 		(unit 1)
 		(exclude_from_sim yes)
@@
 		(fields_autoplaced yes)
 		(property "Reference" "H1"
-			(at 238.76 33.0199 0)
+			(at 219.71 33.0199 0)
 			(effects
 				(font
@@
 		)
 		(property "Value" "MountingHole_Pad"
-			(at 238.76 35.5599 0)
+			(at 219.71 35.5599 0)
 			(effects
 				(font
@@
 		)
 		(property "Footprint" "MountingHole:MountingHole_3.2mm_M3_ISO14580_Pad_TopBottom"
-			(at 236.22 35.56 0)
+			(at 217.17 35.56 0)
 			(effects
 				(font
@@
 		)
 		(property "Datasheet" "~"
-			(at 236.22 35.56 0)
+			(at 217.17 35.56 0)
 			(effects
 				(font
@@
 		)
 		(property "Description" "Mounting Hole with connection"
-			(at 236.22 35.56 0)
+			(at 217.17 35.56 0)
 			(effects
 				(font
@@
 	(symbol
 		(lib_id "power:GND")
-		(at 259.08 38.1 0)
+		(at 240.03 38.1 0)
 		(unit 1)
 		(exclude_from_sim no)
@@
 		(fields_autoplaced yes)
 		(property "Reference" "#PWR09"
-			(at 259.08 44.45 0)
+			(at 240.03 44.45 0)
 			(effects
 				(font
@@
 		)
 		(property "Value" "GND"
-			(at 259.08 43.18 0)
+			(at 240.03 43.18 0)
 			(effects
 				(font
@@
 		)
 		(property "Footprint" ""
-			(at 259.08 38.1 0)
+			(at 240.03 38.1 0)
 			(effects
 				(font
@@
 		)
 		(property "Datasheet" ""
-			(at 259.08 38.1 0)
+			(at 240.03 38.1 0)
 			(effects
 				(font
@@
 		)
 		(property "Description" "Power symbol creates a global label with name \"GND\" , ground"
-			(at 259.08 38.1 0)
+			(at 240.03 38.1 0)
 			(effects
 				(font
@@
 	(symbol
 		(lib_id "Mechanical:MountingHole_Pad")
-		(at 259.08 35.56 0)
+		(at 240.03 35.56 0)
 		(unit 1)
 		(exclude_from_sim yes)
@@
 		(fields_autoplaced yes)
 		(property "Reference" "H2"
-			(at 261.62 33.0199 0)
+			(at 242.57 33.0199 0)
 			(effects
 				(font
@@
 		)
 		(property "Value" "MountingHole_Pad"
-			(at 261.62 35.5599 0)
+			(at 242.57 35.5599 0)
 			(effects
 				(font
@@
 		)
 		(property "Footprint" "MountingHole:MountingHole_3.2mm_M3_ISO14580_Pad_TopBottom"
-			(at 259.08 35.56 0)
+			(at 240.03 35.56 0)
 			(effects
 				(font
@@
 		)
 		(property "Datasheet" "~"
-			(at 259.08 35.56 0)
+			(at 240.03 35.56 0)
 			(effects
 				(font
@@
 		)
 		(property "Description" "Mounting Hole with connection"
-			(at 259.08 35.56 0)
+			(at 240.03 35.56 0)
 			(effects
 				(font
@@
 					(unit 1)
 				)
-			)
-		)
-	)
-	(symbol
-		(lib_id "power:GND")
-		(at 259.08 50.8 0)
-		(unit 1)
-		(exclude_from_sim no)
-		(in_bom yes)
-		(on_board yes)
-		(dnp no)
-		(fields_autoplaced yes)
-		(property "Reference" "#PWR012"
-			(at 259.08 57.15 0)
-			(effects
-				(font
-					(size 1.27 1.27)
-				)
-				(hide yes)
-			)
-		)
-		(property "Value" "GND"
-			(at 259.08 55.88 0)
-			(effects
-				(font
-					(size 1.27 1.27)
-				)
-			)
-		)
-		(property "Footprint" ""
-			(at 259.08 50.8 0)
-			(effects
-				(font
-					(size 1.27 1.27)
-				)
-				(hide yes)
-			)
-		)
-		(property "Datasheet" ""
-			(at 259.08 50.8 0)
-			(effects
-				(font
-					(size 1.27 1.27)
-				)
-				(hide yes)
-			)
-		)
-		(property "Description" "Power symbol creates a global label with name \"GND\" , ground"
-			(at 259.08 50.8 0)
-			(effects
-				(font
-					(size 1.27 1.27)
-				)
-				(hide yes)
-			)
-		)
-		(pin "1"
-		)
-		(instances
-			(project "Module"
-				(path "/34951e98-25fa-4bcc-a56f-5aa93e8633e9"
-					(reference "#PWR012")
-					(unit 1)
-				)

Commit message: Replaced capacitor footprint with EIA-3216
Parts:
- C3, C9: footprint Capacitor_Tantalum_SMD:CP_EIA-3528-15_AVX-H -> Capacitor_Tantalum_SMD:CP_EIA-3216-18_Kemet-A
Changed lines of the file:
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@@
 			)
 		)
-		(property "Footprint" "Capacitor_Tantalum_SMD:CP_EIA-3528-15_AVX-H"
+		(property "Footprint" "Capacitor_Tantalum_SMD:CP_EIA-3216-18_Kemet-A"
 			(at 182.5752 148.59 0)
 			(effects
@@
 			)
 		)
-		(property "Footprint" "Capacitor_Tantalum_SMD:CP_EIA-3528-15_AVX-H"
+		(property "Footprint" "Capacitor_Tantalum_SMD:CP_EIA-3216-18_Kemet-A"
 			(at 196.5452 88.9 0)
 			(effects
